Commit message: simulation working

File: src/mobile_arm_description/description/cyton/cyton_ignition.xacro (robot description, xacro)
@@ -48,9 +48,4 @@
 <robot xmlns:xacro="http://www.ros.org/wiki/xacro">
   <xacro:macro name="cyton_ignition" >
-    <gazebo>
-      <plugin name="ign_ros2_control::IgnitionROS2ControlPlugin" filename="libign_ros2_control-system.so" >
-      <parameters> $(find cyton_bringup)/config/cyton_controller.yaml </parameters>
-      </plugin>
-    </gazebo>
   <ros2_control name="IgnitionSystem" type="system">
     <hardware>

File: src/mobile_arm_description/description/cyton/cyton_macros.urdf.xacro (robot description, xacro)
@@ -8,34 +8,4 @@
             <xacro:cyton_hardware initial_positions_file="$(arg initial_positions_file)"/>
         </xacro:unless>
-        <!-- <material name="blue">
-          <color rgba= "1 0 0 1"/>
-        </material> -->
-        <!-- Initial footprint motor used here -->
-        <!-- <link name="base_footprint">
-                <inertial>
-                    <mass value="2.92"/>
-                    <origin rpy="0 0 0" xyz="-0.025566 -2.88e-05 0.057332"/>
-                    <inertia ixx="0.00782229414331" ixy="-1.56191622996e-05" ixz="-0.00126005738123" iyy="0.0109027971813" iyz="1.08233858202e-05" izz="0.0102355503949"/>
-                  </inertial>
-                <visual>
-                    <origin xyz="0 0 1" rpy="0 0 0" />
-                    <geometry>
-                        <sphere radius="0.001" />
-                    </geometry>
-                    <material name="blue"/>
-                </visual>
-                <collision>
-                    <origin xyz="0 0 1" rpy="0 0 0" />
-                    <geometry>
-                        <sphere radius="0.01" />
-                    </geometry>
-                </collision>
-        </link>
-        <joint name="base_joint" type="fixed">
-                <parent link="base_footprint" />
-                <child link="base_link" />
-                <dynamics damping="0.5" friction="0.5"/>
-                <origin xyz="0.0 0.0 0.0" rpy="0 0 0" />
-        </joint> -->
         <!-- Base of robot here -->
         <link name="arm_base_link">

File: src/mobile_arm_description/description/pioneer3dx/main.xacro (robot description, xacro)
@@ -22,5 +22,10 @@
   <xacro:vehicle_body name="body" parent="base_link"/>
   <!-- differential drive  and joint stage plugin -->
-  <xacro:include filename="${models_dir}/${robot_model}/plugins.xacro"/>
+  <xacro:if value="$(arg use_sim)">
+    <xacro:include filename="${models_dir}/${robot_model}/plugins_ignition.xacro"/>
+  </xacro:if>
+  <xacro:unless value="$(arg use_sim)">
+    <xacro:include filename="${models_dir}/${robot_model}/plugins_hardware.xacro"/>
+  </xacro:unless>
   <xacro:differential_drive    name="$(arg robot_name)"/>
   <xacro:joint_state_publisher name="$(arg robot_name)"/>

File: src/mobile_arm_description/description/pioneer3dx/plugins_ignition.xacro (robot description, xacro)
@@ -33,5 +33,5 @@
     <gazebo>
         <plugin name="ign_ros2_control::IgnitionROS2ControlPlugin" filename="libign_ros2_control-system.so" >
-            <parameters>$(find mobile_arm_bringup)/config/pioneer_control.yaml</parameters>
+            <parameters>$(find mobile_arm_bringup)/config/mobile_arm_controller.yaml</parameters>
         </plugin>
     </gazebo>
