Commit message: default world and sim working

File: src/mobile_arm_description/description/cyton/cyton_macros.urdf copy.xacro (robot description, xacro)
@@ -9,5 +9,5 @@
                     <mesh filename="file://$(arg models_dir)/cyton/meshes/visual/gamma_base.dae" />
                 </geometry>
-                <material name="blue"/>
+                <material name="orange"/>
             </visual>
             <collision>
@@ -17,5 +17,4 @@
                     <!-- <box size="0.1 0.1 0.007" /> -->
                 </geometry>
-                <material name="blue"/>
             </collision>
             <inertial>
@@ -26,4 +25,7 @@
             </inertial>
         </link>
+            <gazebo reference="arm_base_link">
+              <material value="Gazebo/Black"/>
+            </gazebo>
         <!-- First motor located here -->
         <joint name="joint1" type="revolute">
@@ -41,5 +43,5 @@
                     <mesh filename="file://$(arg models_dir)/cyton/meshes/visual/link1.dae" />
                 </geometry>
-                <material name="blue"/>
+                <material name="orange"/>
             </visual>
             <collision>
@@ -56,4 +58,7 @@
             </inertial>
         </link>
+            <gazebo reference="link1">
+              <material value="Gazebo/Black"/>
+            </gazebo>
         <!-- Second motor located here -->
         <joint name="joint2" type="revolute">
@@ -71,5 +76,5 @@
                     <mesh filename="file://$(arg models_dir)/cyton/meshes/visual/link2.dae" />
                 </geometry>
-                <material name="blue"/>
+                <material name="orange"/>
             </visual>
             <collision>
@@ -86,4 +91,7 @@
             </inertial>
         </link>
+            <gazebo reference="link2">
+              <material value="Gazebo/Black"/>
+            </gazebo>
         <!-- Third motor located here -->
         <joint name="joint3" type="revolute">
@@ -102,5 +110,5 @@
                     <mesh filename="file://$(arg models_dir)/cyton/meshes/visual/link3.dae" />
                 </geometry>
-                <material name="blue"/>
+                <material name="orange"/>
             </visual>
             <collision>
@@ -118,4 +126,7 @@
             </inertial>
         </link>
+            <gazebo reference="link3">
+              <material value="Gazebo/Black"/>
+            </gazebo>
         <!-- Fourth motor located here -->
         <joint name="joint4" type="revolute">
@@ -134,5 +145,5 @@
                     <mesh filename="file://$(arg models_dir)/cyton/meshes/visual/link4.dae" />
                 </geometry>
-                <material name="blue"/>
+                <material name="orange"/>
             </visual>
             <collision>
@@ -150,4 +161,7 @@
             </inertial>
         </link>
+            <gazebo reference="link4">
+              <material value="Gazebo/Black"/>
+            </gazebo>
         <!-- Fifth motor located here -->
         <joint name="joint5" type="revolute">
@@ -165,5 +179,5 @@
                     <mesh filename="file://$(arg models_dir)/cyton/meshes/visual/link5.dae" />
                 </geometry>
-                <material name="blue"/>
+                <material name="orange"/>
             </visual>
             <collision>
@@ -181,4 +195,7 @@
             </inertial>
         </link>
+            <gazebo reference="link5">
+              <material value="Gazebo/Black"/>
+            </gazebo>
         <!-- Sixth motor located here -->
         <joint name="joint6" type="revolute">
@@ -196,5 +213,5 @@
                     <mesh filename="file://$(arg models_dir)/cyton/meshes/visual/link6.dae" />
                 </geometry>
-                <material name="blue"/>
+                <material name="orange"/>
             </visual>
             <collision>
@@ -212,4 +229,7 @@
             </inertial>
         </link>
+            <gazebo reference="link6">
+              <material value="Gazebo/Black"/>
+            </gazebo>
         <!-- Seventh motor located here -->
         <joint name="joint7" type="revolute">
@@ -227,5 +247,5 @@
                     <mesh filename="file://$(arg models_dir)/cyton/meshes/visual/link7.dae" />
                 </geometry>
-                <material name="blue"/>
+                <material name="orange"/>
             </visual>
             <collision>
@@ -237,5 +257,5 @@
             </collision>
             <inertial>
-                <mass value="0.15" />
+                <mass value="0.01" />
                 <origin rpy="0 0 0" xyz="0 0 0" />
                 <inertia  ixx="0.0015572863522148085" ixy="0" ixz="0"
@@ -243,7 +263,67 @@
             </inertial>
         </link>
-        <!-- Eighth motor located here -->
+            <gazebo reference="link7">
+              <material value="Gazebo/Black"/>
+            </gazebo>
+        <joint name="gripper_spacer_joint" type="fixed">
+            <parent link="link7" />
+            <child link="gripper_spacer" />
+            <origin xyz="0.0 0.0 0.048" rpy="0 0 0" />
+        </joint>
+        <link name="gripper_spacer">
+            <visual>
+                <origin xyz="-0.0125 -0.0225 0.0" rpy="-1.5708 0 0" />
+                <geometry>
+                    <mesh filename="file://$(arg models_dir)/cyton/meshes/visual/gripper_spacer.dae"/>
+                </geometry>
+                <material name="orange"/>
+            </visual>
+            <collision>
+                <origin xyz="-0.0125 -0.0225 0.0" rpy="-1.5708 0 0" />
+                <geometry>
+                    <mesh filename="file://$(arg models_dir)/cyton/meshes/collision/gripper_spacer.stl"/>
+                </geometry>
+            </collision>
+            <inertial>
+                <mass value="0.01" />
+                <origin rpy="0 0 0" xyz="0 0 0" />
+                <inertia  ixx="0.00011683333934843555" ixy="0" ixz="0"
+                    iyy="9.527084112726167e-05" iyz="0" izz="5.193749979697169e-05" />
+            </inertial>
+        </link>
+            <gazebo reference="gripper_spacer">
+              <material value="Gazebo/Black"/>
+            </gazebo>
+        <joint name="gripper_base_joint" type="fixed">
+            <parent link="gripper_spacer" />
+            <child link="gripper_base" />
+            <origin xyz="0.0 0.0 0.05" rpy="0 0 0" />
+        </joint>
+        <link name="gripper_base">
+            <visual>
+                <origin xyz="0.0185 0.035 0.0" rpy="-1.5708 0 0" />
+                <geometry>
+                    <mesh filename="file://$(arg models_dir)/cyton/meshes/visual/gripper_base.dae"/>
+                </geometry>
+                <material name="orange"/>
+            </visual>
+            <collision>
+                <origin xyz="0.0185 0.035 0.0" rpy="-1.5708 0 0" />
+                <geometry>
+                    <mesh filename="file://$(arg models_dir)/cyton/meshes/collision/gripper_base.stl"/>
+                </geometry>
+            </collision>
+            <inertial>
+                <mass value="0.02" />
+                <origin rpy="0 0 0" xyz="0 0 0" />
+                <inertia  ixx="0.00011683333934843555" ixy="0" ixz="0"
+                    iyy="9.527084112726167e-05" iyz="0" izz="5.193749979697169e-05" />
+            </inertial>
+        </link>
+            <gazebo reference="gripper_base">
+              <material value="Gazebo/Black"/>
+            </gazebo>
         <joint name="joint8" type="prismatic">
-            <parent link="link7" />
+            <parent link="gripper_base" />
             <child link="link8" />
             <origin xyz="-0.02131 0.00485 0.077225" rpy="0 0 0" />
@@ -252,24 +332,16 @@
             <axis xyz="1 0 0" />
         </joint>
-        <!-- <joint name="joint8" type="prismatic">
-            <parent link="joint7" />
-            <child link="joint8" />
-            <origin xyz="-0.05331 0.00485 0.077225" rpy="0 0 0" />
-            <dynamics damping="0.5" friction="0.5"/>
-            <limit lower="-0.001" upper="0.017" effort="100.0" velocity="1.0" />
-            <axis xyz="1 0 0" />
-        </joint> -->
         <link name="link8">
             <visual>
-                <origin xyz="0 0.0 -0.035" rpy="0 0 0" />
-                <geometry>
-                    <mesh filename="file://$(arg models_dir)/cyton/meshes/visual/link8.dae" scale="1.0 1.0 2.0"/>
-                </geometry>
-                <material name="blue"/>
-            </visual>
-            <collision>
-                <origin xyz="0 0.0 -0.035" rpy="0 0 0" />
-                <geometry>
-                    <mesh filename="file://$(arg models_dir)/cyton/meshes/collision/link8.stl" scale="1.0 1.0 2.0"/>
+                <origin xyz="0 0.0185 -0.035" rpy="0 0 3.14" />
+                <geometry>
+                    <mesh filename="file://$(arg models_dir)/cyton/meshes/visual/finger.dae"/>
+                </geometry>
+                <material name="orange"/>
+            </visual>
+            <collision>
+                <origin xyz="0 0.0185 -0.035" rpy="0 0 3.14" />
+                <geometry>
+                    <mesh filename="file://$(arg models_dir)/cyton/meshes/collision/finger.stl"/>
                 </geometry>
             </collision>
@@ -281,7 +353,9 @@
             </inertial>
         </link>
-        <!-- Eighth motor located here -->
+            <gazebo reference="link8">
+              <material value="Gazebo/Black"/>
+            </gazebo>
         <joint name="joint9" type="prismatic">
-            <parent link="link7" />
+            <parent link="gripper_base" />
             <child link="link9" />
             <origin xyz="0.0178 0.00485 0.077225" rpy="0 0 0" />
@@ -295,12 +369,12 @@
                 <origin xyz="0 0 -0.035" rpy="0 0 0" />
                 <geometry>
-                    <mesh filename="file://$(arg models_dir)/cyton/meshes/visual/link9.dae" scale="1.0 1.0 2.0"/>
-                </geometry>
-                <material name="blue"/>
+                    <mesh filename="file://$(arg models_dir)/cyton/meshes/visual/finger.dae"/>
+                </geometry>
+                <material name="orange"/>
             </visual>
             <collision>
                 <origin xyz="0 0 -0.035" rpy="0 0 0" />
                 <geometry>
-                    <mesh filename="file://$(arg models_dir)/cyton/meshes/collision/link9.stl" scale="1.0 1.0 2.0"/>
+                    <mesh filename="file://$(arg models_dir)/cyton/meshes/collision/finger.stl"/>
                 </geometry>
             </collision>
@@ -312,4 +386,7 @@
             </inertial>
         </link>
+            <gazebo reference="link9">
+              <material value="Gazebo/Black"/>
+            </gazebo>
         <!-- Dummy joint/link to prevent error with mimic joint -->
         <joint name="joint9_mimic" type="fixed">

File: src/mobile_arm_description/description/pioneer3dx/body/body.xacro (robot description, xacro)
@@ -17,5 +17,5 @@
     <xacro:pioneer_sonar name="sonar" parent="${name}" xyz="0.109 0 0.15" rpy="0 0 0"/>
     <!-- Akku0 -->
-    <xacro:pioneer_battery_block name="battery0" parent="${name}" x="-0.14" y="0.00"  z="${0.13-0.068}" mass="2.5" />
+    <xacro:pioneer_battery_block name="battery0" parent="${name}" x="-0.14" y="0.00"  z="${0.13-0.068}" mass="5.5" />
     <!-- Wheels -->
     <!-- <xacro:property name="contact_data">
