Commit message: urdfs done

File: src/mobile_arm_description/description/cyton/cyton_macros.urdf.xacro (robot description, xacro)
@@ -8,10 +8,9 @@
             <xacro:cyton_hardware initial_positions_file="$(arg initial_positions_file)"/>
         </xacro:unless>
-        <material name="blue">
+        <!-- <material name="blue">
           <color rgba= "1 0 0 1"/>
-        </material>
+        </material> -->
         <!-- Initial footprint motor used here -->
-        <link name="base_footprint">
-                <!-- ZMIENIĆ!!! -->
+        <!-- <link name="base_footprint">
                 <inertial>
                     <mass value="2.92"/>
@@ -38,7 +37,7 @@
                 <dynamics damping="0.5" friction="0.5"/>
                 <origin xyz="0.0 0.0 0.0" rpy="0 0 0" />
-        </joint>
+        </joint> -->
         <!-- Base of robot here -->
-        <link name="base_link">
+        <link name="arm_base_link">
             <visual>
                 <origin xyz="0 0 0" rpy="0 0 0" />
@@ -65,5 +64,5 @@
         <!-- First motor located here -->
         <joint name="joint1" type="revolute">
-            <parent link="base_link" />
+            <parent link="arm_base_link" />
             <child link="link1" />
             <origin xyz="0 0 0.05315" rpy="0 0 0" />
@@ -352,5 +351,5 @@
         <!-- Dummy joint/link to prevent error with mimic joint -->
         <joint name="joint9_mimic" type="fixed">
-            <parent link="world" />
+            <parent link="arm_base_link" />
             <child link="dummy_mimic_fix" />
         </joint>

File: src/mobile_arm_description/description/cyton/main.xacro (robot description, xacro)
@@ -8,5 +8,5 @@
         <origin xyz="${xyz}" rpy="${rpy}"/>
         <parent link="${parent}"/>
-        <child link="base_footprint"/>
+        <child link="arm_base_link"/>
     </joint>
     <xacro:include filename="$(arg models_dir)/cyton/cyton_macros.urdf.xacro" />

File: src/mobile_arm_description/description/pioneer3dx/body/body.xacro (robot description, xacro)
@@ -1,5 +1,5 @@
 <?xml version="1.0"?>
 <robot xmlns:xacro="http://ros.org/wiki/xacro">
-  <xacro:include filename="$(find pioneer_description)/description/inertia_tensors.xacro"/>
+  <xacro:include filename="$(find mobile_arm_description)/description/inertia_tensors.xacro"/>
   <xacro:include filename="chassis.xacro"/>
   <xacro:include filename="wheel.xacro"/>

File: src/mobile_arm_description/description/pioneer3dx/main.xacro (robot description, xacro)
@@ -29,5 +29,5 @@
   <xacro:laser name="laser0" parent="top" namespace="${namespace}" topic_name="$(arg laser0_topic)" frame_name="laser0" xyz="0.15 0.0 0.06" rpy="0 0 0" driver="$(arg laser0_driver)" visualize="$(arg laser0_visualize)"/>
   <!-- Arm -->
-  <xacro:include filename="${models_dir}/${arm_model}/urdf/main.xacro" />
-  <xacro:arm name="cyton" parent="top" xyz="0.0 0.0 0.0" rpy="0 0 0" use_sim="$(use_sim)"/>
+  <xacro:include filename="${models_dir}/${arm_model}/main.xacro" />
+  <xacro:arm name="cyton" parent="top" xyz="0.0 0.0 0.0" rpy="0 0 0" use_sim="$(arg use_sim)"/>
 </robot>

File: src/mobile_arm_description/description/pioneer3dx/plugins.xacro (robot description, xacro)
@@ -33,5 +33,5 @@
     <gazebo>
         <plugin name="ign_ros2_control::IgnitionROS2ControlPlugin" filename="libign_ros2_control-system.so" >
-            <parameters>$(find pioneer_bringup)/config/pioneer_control.yaml</parameters>
+            <parameters>$(find mobile_arm_bringup)/config/pioneer_control.yaml</parameters>
         </plugin>
     </gazebo>

Commit message: moveit working fine

File: src/mobile_arm_description/description/cyton/cyton_macros.urdf.xacro (robot description, xacro)
@@ -2,10 +2,4 @@
 <robot xmlns:xacro="http://www.ros.org/wiki/xacro">
     <xacro:macro name="cyton_robot">
-        <xacro:if value="$(arg use_sim)">
-            <xacro:cyton_ignition />
-        </xacro:if>
-        <xacro:unless value="$(arg use_sim)">
-            <xacro:cyton_hardware initial_positions_file="$(arg initial_positions_file)"/>
-        </xacro:unless>
         <!-- Base of robot here -->
         <link name="arm_base_link">

File: src/mobile_arm_description/description/cyton/main.xacro (robot description, xacro)
@@ -2,5 +2,5 @@
 <robot xmlns:xacro="http://www.ros.org/wiki/xacro" name="cyton">
   <xacro:macro name="arm" params="name parent use_sim xyz rpy" >
-    <xacro:arg name="use_sim" default="False"/>
+    <xacro:arg name="use_sim" default="True"/>
     <xacro:arg name="initial_positions_file" default="$(find mobile_arm_moveit)/config/initial_positions.yaml" />
     <joint name="${parent}_${name}_joint" type="fixed">
@@ -11,10 +11,4 @@
     </joint>
     <xacro:include filename="$(arg models_dir)/cyton/cyton_macros.urdf.xacro" />
-    <xacro:if value="$(arg use_sim)">
-      <xacro:include filename="$(arg models_dir)/cyton/cyton_ignition.xacro" />
-    </xacro:if>
-    <xacro:unless value="$(arg use_sim)">
-      <xacro:include filename="$(arg models_dir)/cyton/cyton.hardware.xacro" />
-    </xacro:unless>
     <xacro:cyton_robot/>
   </xacro:macro>

File: src/mobile_arm_description/description/pioneer3dx/main.xacro (robot description, xacro)
@@ -10,5 +10,5 @@
   <xacro:arg name="laser0_visualize" default="true"/>
   <xacro:arg name="laser0_driver"    default="gpu"/>
-  <xacro:arg name="use_sim"          default="false"/>
+  <xacro:arg name="use_sim"          default="true"/>
   <xacro:property name="models_dir"    value="$(arg models_dir)"/>
   <xacro:property name="namespace"    value="$(arg namespace)"/>
@@ -22,12 +22,12 @@
   <xacro:vehicle_body name="body" parent="base_link"/>
   <!-- differential drive  and joint stage plugin -->
+    <xacro:include filename="${models_dir}/${robot_model}/plugins_ignition.xacro"/>
+    <xacro:include filename="${models_dir}/${robot_model}/plugins_hardware.xacro"/>
   <xacro:if value="$(arg use_sim)">
-    <xacro:include filename="${models_dir}/${robot_model}/plugins_ignition.xacro"/>
+    <xacro:plugins_ignition />
   </xacro:if>
   <xacro:unless value="$(arg use_sim)">
-    <xacro:include filename="${models_dir}/${robot_model}/plugins_hardware.xacro"/>
+    <xacro:plugins_hardware initial_positions_file="$(arg initial_positions_file)"/>
   </xacro:unless>
-  <xacro:differential_drive    name="$(arg robot_name)"/>
-  <xacro:joint_state_publisher name="$(arg robot_name)"/>
   <!-- Laser -->
   <xacro:include filename="${models_dir}/${laser_model}/main.xacro"/>

File: src/mobile_arm_description/description/pioneer3dx/plugins_hardware.xacro (robot description, xacro)
@@ -1,6 +1,5 @@
 <?xml version="1.0"?>
-<robot xmlns:xacro="http://www.ros.org/wiki/xacro">
-      <!-- <xacro:macro name="cyton_hardware"> -->
-      <xacro:macro name="cyton_hardware" params="initial_positions_file">
+<robot xmlns:xacro="http://ros.org/wiki/xacro">
+    <xacro:macro name="plugins_hardware" params="initial_positions_file">
       <xacro:property name="initial_positions" value="${xacro.load_yaml(initial_positions_file)['initial_positions']}"/>
         <ros2_control name="DynamixelHardware" type="system">
@@ -78,3 +77,4 @@
         </ros2_control>
     </xacro:macro>
+<!-- insert ros2 hardware controllers here -->
 </robot>

File: src/mobile_arm_description/description/pioneer3dx/plugins_ignition.xacro (robot description, xacro)
@@ -1,54 +1,146 @@
 <?xml version="1.0"?>
 <robot xmlns:xacro="http://ros.org/wiki/xacro">
-  <xacro:macro name="differential_drive" params="name">
-    <ros2_control name="IgnitionSystem" type="system">
-        <hardware>
-          <plugin>ign_ros2_control/IgnitionSystem</plugin>
-        </hardware>
-        <joint name="left_wheel_joint">
-            <command_interface name="velocity">
-                <param name="min">-10</param>
-                <param name="max">10</param>
+  <xacro:macro name="plugins_ignition">
+      <ros2_control name="IgnitionSystem" type="system">
+          <hardware>
+            <plugin>ign_ros2_control/IgnitionSystem</plugin>
+          </hardware>
+          <joint name="left_wheel_joint">
+              <command_interface name="velocity">
+                  <param name="min">-10</param>
+                  <param name="max">10</param>
+              </command_interface>
+              <state_interface name="velocity"/>
+              <state_interface name="position"/>
+          </joint>
+          <joint name="right_wheel_joint">
+              <command_interface name="velocity">
+                  <param name="min">-10</param>
+                  <param name="max">10</param>
+              </command_interface>
+              <state_interface name="velocity"/>
+              <state_interface name="position"/>
+          </joint>
+          <joint name="swivel_joint">
+              <state_interface name="velocity"/>
+              <state_interface name="position"/>
+          </joint>
+          <joint name="swivel_wheel_joint">
+              <state_interface name="velocity"/>
+              <state_interface name="position"/>
+          </joint>
+          <!-- cyton_joint1 -->
+          <joint name="joint1">
+            <!-- <param name="initial_position">0.0</param> -->
+            <command_interface name="position">
+              <param name="min">-2.8973</param>
+              <param name="max">2.8973</param>
             </command_interface>
+            <state_interface name="position"/>
             <state_interface name="velocity"/>
+            <state_interface name="effort"/>
+          </joint>
+          <!-- cyton_joint2 -->
+          <joint name="joint2">
+            <!-- <param name="initial_position">-0.785</param> -->
+            <command_interface name="position">
+              <param name="min">-1.7628</param>
+              <param name="max">1.7628</param>
+            </command_interface>
             <state_interface name="position"/>
+            <state_interface name="velocity"/>
+            <state_interface name="effort"/>
+          </joint>
+          <!-- cyton_joint3 -->
+          <joint name="joint3">
+            <!-- <param name="initial_position">0.0</param> -->
+            <command_interface name="position">
+              <param name="min">-2.8973</param>
+              <param name="max">2.8973</param>
+            </command_interface>
+            <state_interface name="position"/>
+            <state_interface name="velocity"/>
+            <state_interface name="effort"/>
+          </joint>
+          <!-- cyton_joint4 -->
+          <joint name="joint4">
+            <!-- <param name="initial_position">-2.356</param> -->
+            <command_interface name="position">
+              <param name="min">-3.0718</param>
+              <param name="max">0.0698</param>
+            </command_interface>
+            <state_interface name="position"/>
+            <state_interface name="velocity"/>
+            <state_interface name="effort"/>
+          </joint>
+          <!-- cyton_joint5 -->
+          <joint name="joint5">
+            <!-- <param name="initial_position">0.0</param> -->
+            <command_interface name="position">
+              <param name="min">-2.8973</param>
+              <param name="max">2.8973</param>
+            </command_interface>
+            <state_interface name="position"/>
+            <state_interface name="velocity"/>
+            <state_interface name="effort"/>
+          </joint>
+                <!-- cyton_joint7 -->
+          <joint name="joint6">
+            <!-- <param name="initial_position">0.785</param> -->
+            <command_interface name="position">
+              <param name="min">-3.15</param> <!-- ** -3.935 -->
+              <param name="max">3.15</param> <!-- ** 2.365 -->
+            </command_interface>
+            <state_interface name="position"/>
+            <state_interface name="velocity"/>
+            <state_interface name="effort"/>
+          </joint>
+          <!-- cyton_joint6 -->
+          <joint name="joint7">
+            <!-- <param name="initial_position">1.5708</param> -->
+            <command_interface name="position">
+              <param name="min">-0.0175</param> <!-- ** -1.5883 -->
+              <param name="max">3.7525</param> <!-- ** 2.1817 -->
+            </command_interface>
+            <state_interface name="position"/>
+            <state_interface name="velocity"/>
+            <state_interface name="effort"/>
+          </joint>
+          <!-- cyton_joint7 -->
+          <joint name="joint8">
+            <!-- <param name="initial_position">0.785</param> -->
+            <command_interface name="position">
+              <param name="min">-3.15</param> <!-- ** -3.935 -->
+              <param name="max">3.15</param> <!-- ** 2.365 -->
+            </command_interface>
+            <state_interface name="position"/>
+            <state_interface name="velocity"/>
+            <state_interface name="effort"/>
+          </joint>
+        <joint name="joint9">
+          <param name="mimic">joint8</param>
+          <param name="multiplier">-1</param>
+          <command_interface name="position"></command_interface>
+          <state_interface name="position"></state_interface>
         </joint>
-        <joint name="right_wheel_joint">
-            <command_interface name="velocity">
-                <param name="min">-10</param>
-                <param name="max">10</param>
-            </command_interface>
-            <state_interface name="velocity"/>
-            <state_interface name="position"/>
-        </joint>
-        <joint name="swivel_joint">
-            <state_interface name="velocity"/>
-            <state_interface name="position"/>
-        </joint>
-        <joint name="swivel_wheel_joint">
-            <state_interface name="velocity"/>
-            <state_interface name="position"/>
-        </joint>
-    </ros2_control>
-    <gazebo>
-        <plugin name="ign_ros2_control::IgnitionROS2ControlPlugin" filename="libign_ros2_control-system.so" >
-            <parameters>$(find mobile_arm_bringup)/config/mobile_arm_controller.yaml</parameters>
-        </plugin>
-    </gazebo>
-  </xacro:macro>
-  <xacro:macro name="joint_state_publisher" params="name">
-    <gazebo>
-    <plugin name="gazebo_ros_joint_state_publisher"
-        filename="libgazebo_ros_joint_state_publisher.so">
-      <ros>
-        <remapping>joint_states:=joint_states</remapping>
-      </ros>
-      <update_rate>10</update_rate>
-      <joint_name>left_wheel_joint</joint_name>
-      <joint_name>right_wheel_joint</joint_name>
-      <joint_name>swivel_joint</joint_name>
-      <joint_name>swivel_wheel_joint</joint_name>
-    </plugin>
-    </gazebo>
+      </ros2_control>
+      <gazebo>
+          <plugin name="ign_ros2_control::IgnitionROS2ControlPlugin" filename="libign_ros2_control-system.so" >
+              <parameters>$(find mobile_arm_bringup)/config/mobile_arm_controller.yaml</parameters>
+          </plugin>
+      </gazebo>
+      <!-- <gazebo>
+      <plugin name="gazebo_ros_joint_state_publisher"
+          filename="libgazebo_ros_joint_state_publisher.so">
+        <ros>
+          <remapping>joint_states:=joint_states</remapping>
+        </ros>
+        <update_rate>10</update_rate>
+        <joint_name>left_wheel_joint</joint_name>
+        <joint_name>right_wheel_joint</joint_name>
+        <joint_name>swivel_joint</joint_name>
+        <joint_name>swivel_wheel_joint</joint_name>
+      </plugin>
+      </gazebo>     -->
   </xacro:macro>
 </robot>

Commit message: fingers position fixed

File: src/mobile_arm_description/description/cyton/cyton_macros.urdf.xacro (robot description, xacro)
@@ -20,5 +20,5 @@
             </collision>
             <inertial>
-                <mass value="0.2" />
+                <mass value="0.15" />
                 <origin rpy="0 0 0" xyz="0 0 0" />
                 <inertia ixx="1.1027" iyy="1.1027" izz="1.1027"
@@ -50,5 +50,5 @@
             </collision>
             <inertial>
-                <mass value="5.0" />
+                <mass value="0.15" />
                 <origin rpy="0 0 0" xyz="0 0 0" />
                 <inertia  ixx="0.011208614136379117" ixy="0" ixz="0"
@@ -80,5 +80,5 @@
             </collision>
             <inertial>
-                <mass value="2.0" />
+                <mass value="0.15" />
                 <origin rpy="0 0 0" xyz="0 0 0" />
                 <inertia  ixx="0.004978331673653838" ixy="0" ixz="0"
@@ -112,5 +112,5 @@
             </collision>
             <inertial>
-                <mass value="0.2" />
+                <mass value="0.15" />
                 <origin rpy="0 0 0" xyz="0 0 0" />
                 <inertia  ixx="0.004185745441913727" ixy="0" ixz="0"
@@ -144,5 +144,5 @@
             </collision>
             <inertial>
-                <mass value="0.2" />
+                <mass value="0.15" />
                 <origin rpy="0 0 0" xyz="0 0 0" />
                 <inertia  ixx="0.0002991427484832406" ixy="0" ixz="0"
@@ -175,5 +175,5 @@
             </collision>
             <inertial>
-                <mass value="0.2" />
+                <mass value="0.15" />
                 <origin rpy="0 0 0" xyz="0 0 0" />
                 <inertia  ixx="0.004619866095305994" ixy="0" ixz="0"
@@ -206,5 +206,5 @@
             </collision>
             <inertial>
-                <mass value="0.2" />
+                <mass value="0.15" />
                 <origin rpy="0 0 0" xyz="0 0 0" />
                 <inertia  ixx="0.002306163215052582" ixy="0" ixz="0"
@@ -237,5 +237,5 @@
             </collision>
             <inertial>
-                <mass value="0.2" />
+                <mass value="0.15" />
                 <origin rpy="0 0 0" xyz="0 0 0" />
                 <inertia  ixx="0.0015572863522148085" ixy="0" ixz="0"
@@ -262,5 +262,5 @@
         <link name="link8">
             <visual>
-                <origin xyz="0 0 -0.035" rpy="0 0 3.14" />
+                <origin xyz="0 0.0185 -0.035" rpy="0 0 3.14" />
                 <geometry>
                     <mesh filename="file://$(arg models_dir)/cyton/meshes/visual/joint9_stretched.dae"/>
@@ -269,5 +269,5 @@
             </visual>
             <collision>
-                <origin xyz="0 0 -0.035" rpy="0 0 3.14" />
+                <origin xyz="0 0.0185 -0.035" rpy="0 0 3.14" />
                 <geometry>
                     <mesh filename="file://$(arg models_dir)/cyton/meshes/collision/joint9_stretched.stl"/>
