Commit message: links names changed and fingers position fis

File: src/mobile_arm_description/description/cyton/cyton_macros.urdf.xacro (robot description, xacro)
@@ -39,5 +39,5 @@
                 <origin xyz="0 0 0" rpy="1.5708 0 3.14159" />
                 <geometry>
-                    <mesh filename="file://$(arg models_dir)/cyton/meshes/visual/joint1.dae" />
+                    <mesh filename="file://$(arg models_dir)/cyton/meshes/visual/link1.dae" />
                 </geometry>
                 <material name="blue"/>
@@ -46,5 +46,5 @@
                 <origin xyz="0 0 0" rpy="1.5708 0 3.14159" />
                 <geometry>
-                    <mesh filename="file://$(arg models_dir)/cyton/meshes/collision/joint1.stl" />
+                    <mesh filename="file://$(arg models_dir)/cyton/meshes/collision/link1.stl" />
                 </geometry>
             </collision>
@@ -69,5 +69,5 @@
                 <origin xyz="0.028 0 0" rpy="0 1.5708 0" />
                 <geometry>
-                    <mesh filename="file://$(arg models_dir)/cyton/meshes/visual/joint2.dae" />
+                    <mesh filename="file://$(arg models_dir)/cyton/meshes/visual/link2.dae" />
                 </geometry>
                 <material name="blue"/>
@@ -76,5 +76,5 @@
                 <origin xyz="0.028 0 0" rpy="0 1.5708 0" />
                 <geometry>
-                    <mesh filename="file://$(arg models_dir)/cyton/meshes/collision/joint2.stl" />
+                    <mesh filename="file://$(arg models_dir)/cyton/meshes/collision/link2.stl" />
                 </geometry>
             </collision>
@@ -100,5 +100,5 @@
                 <origin xyz="0 0 0" rpy="0 0 3.92699" />
                 <geometry>
-                    <mesh filename="file://$(arg models_dir)/cyton/meshes/visual/joint3.dae" />
+                    <mesh filename="file://$(arg models_dir)/cyton/meshes/visual/link3.dae" />
                 </geometry>
                 <material name="blue"/>
@@ -107,5 +107,5 @@
                 <origin xyz="0 0 0" rpy="0 0 3.92699" />
                 <geometry>
-                    <mesh filename="file://$(arg models_dir)/cyton/meshes/collision/joint3.stl" />
+                    <mesh filename="file://$(arg models_dir)/cyton/meshes/collision/link3.stl" />
                     <!-- <sphere radius="0.001" /> -->
                 </geometry>
@@ -132,5 +132,5 @@
                 <origin xyz="0.027 0 0" rpy="1.5708 0 1.5708" />
                 <geometry>
-                    <mesh filename="file://$(arg models_dir)/cyton/meshes/visual/joint4.dae" />
+                    <mesh filename="file://$(arg models_dir)/cyton/meshes/visual/link4.dae" />
                 </geometry>
                 <material name="blue"/>
@@ -139,5 +139,5 @@
                 <origin xyz="0.027 0 0" rpy="1.5708 0 1.5708" />
                 <geometry>
-                    <mesh filename="file://$(arg models_dir)/cyton/meshes/collision/joint4.stl" />
+                    <mesh filename="file://$(arg models_dir)/cyton/meshes/collision/link4.stl" />
                     <!-- <sphere radius="0.001" /> -->
                 </geometry>
@@ -163,5 +163,5 @@
                 <origin xyz="0 0 0" rpy="1.5708 0 0" />
                 <geometry>
-                    <mesh filename="file://$(arg models_dir)/cyton/meshes/visual/joint5.dae" />
+                    <mesh filename="file://$(arg models_dir)/cyton/meshes/visual/link5.dae" />
                 </geometry>
                 <material name="blue"/>
@@ -170,5 +170,5 @@
                 <origin xyz="0 0 0" rpy="1.5708 0 0" />
                 <geometry>
-                    <mesh filename="file://$(arg models_dir)/cyton/meshes/collision/joint5.stl" />
+                    <mesh filename="file://$(arg models_dir)/cyton/meshes/collision/link5.stl" />
                     <!-- <sphere radius="0.001" /> -->
                 </geometry>
@@ -194,5 +194,5 @@
                 <origin xyz="0.027 0 0" rpy="1.5708 0 1.5708" />
                 <geometry>
-                    <mesh filename="file://$(arg models_dir)/cyton/meshes/visual/joint6.dae" />
+                    <mesh filename="file://$(arg models_dir)/cyton/meshes/visual/link6.dae" />
                 </geometry>
                 <material name="blue"/>
@@ -201,5 +201,5 @@
                 <origin xyz="0.027 0 0" rpy="1.5708 0 1.5708" />
                 <geometry>
-                    <mesh filename="file://$(arg models_dir)/cyton/meshes/collision/joint6.stl" />
+                    <mesh filename="file://$(arg models_dir)/cyton/meshes/collision/link6.stl" />
                     <!-- <sphere radius="0.001" /> -->
                 </geometry>
@@ -225,5 +225,5 @@
                 <origin xyz="0 0 0" rpy="0 3.14159 1.5708" />
                 <geometry>
-                    <mesh filename="file://$(arg models_dir)/cyton/meshes/visual/joint7.dae" />
+                    <mesh filename="file://$(arg models_dir)/cyton/meshes/visual/link7.dae" />
                 </geometry>
                 <material name="blue"/>
@@ -232,5 +232,5 @@
                 <origin xyz="0 0 0" rpy="0 3.14159 1.5708" />
                 <geometry>
-                    <mesh filename="file://$(arg models_dir)/cyton/meshes/collision/joint7.stl" />
+                    <mesh filename="file://$(arg models_dir)/cyton/meshes/collision/link7.stl" />
                     <!-- <sphere radius="0.001" /> -->
                 </geometry>
@@ -264,5 +264,5 @@
                 <origin xyz="0 0.0185 -0.035" rpy="0 0 3.14" />
                 <geometry>
-                    <mesh filename="file://$(arg models_dir)/cyton/meshes/visual/joint9_stretched.dae"/>
+                    <mesh filename="file://$(arg models_dir)/cyton/meshes/visual/link9.dae"/>
                 </geometry>
                 <material name="blue"/>
@@ -271,5 +271,5 @@
                 <origin xyz="0 0.0185 -0.035" rpy="0 0 3.14" />
                 <geometry>
-                    <mesh filename="file://$(arg models_dir)/cyton/meshes/collision/joint9_stretched.stl"/>
+                    <mesh filename="file://$(arg models_dir)/cyton/meshes/collision/link9.stl"/>
                 </geometry>
             </collision>
@@ -296,5 +296,5 @@
                 <origin xyz="0 0 -0.035" rpy="0 0 0" />
                 <geometry>
-                    <mesh filename="file://$(arg models_dir)/cyton/meshes/visual/joint9_stretched.dae"/>
+                    <mesh filename="file://$(arg models_dir)/cyton/meshes/visual/link9.dae"/>
                 </geometry>
                 <material name="blue"/>
@@ -303,5 +303,5 @@
                 <origin xyz="0 0 -0.035" rpy="0 0 0" />
                 <geometry>
-                    <mesh filename="file://$(arg models_dir)/cyton/meshes/collision/joint9_stretched.stl"/>
+                    <mesh filename="file://$(arg models_dir)/cyton/meshes/collision/link9.stl"/>
                 </geometry>
             </collision>

Commit message: work in progress

File: src/mobile_arm_description/description/cyton/cyton_macros.urdf.xacro (robot description, xacro)
@@ -249,5 +249,5 @@
             <origin xyz="-0.02131 0.00485 0.077225" rpy="0 0 0" />
             <dynamics damping="0.5" friction="0.5"/>
-            <limit lower="-0.002" upper="0.018" effort="0.1" velocity="1.0" />
+            <limit lower="-0.002" upper="0.018" effort="100.0" velocity="1.0" />
             <axis xyz="1 0 0" />
         </joint>
@@ -287,5 +287,5 @@
             <origin xyz="0.0178 0.00485 0.077225" rpy="0 0 0" />
             <dynamics damping="0.5" friction="0.5"/>
-            <limit lower="-0.018" upper="0.002" effort="0.1" velocity="1.0" />
+            <limit lower="-0.018" upper="0.002" effort="100.0" velocity="1.0" />
             <mimic joint="joint8" multiplier="-1"/>
             <axis xyz="1 0 0" />

Commit message: cleaning

File: src/mobile_arm_description/description/cyton/cyton_macros.urdf.xacro (robot description, xacro)
@@ -9,5 +9,5 @@
                     <mesh filename="file://$(arg models_dir)/cyton/meshes/visual/gamma_base.dae" />
                 </geometry>
-                <material name="blue"/>
+                <material name="TopBlack"/>
             </visual>
             <collision>
@@ -17,5 +17,5 @@
                     <!-- <box size="0.1 0.1 0.007" /> -->
                 </geometry>
-                <material name="blue"/>
+                <material name="TopBlack"/>
             </collision>
             <inertial>
@@ -41,5 +41,5 @@
                     <mesh filename="file://$(arg models_dir)/cyton/meshes/visual/link1.dae" />
                 </geometry>
-                <material name="blue"/>
+                <material name="TopBlack"/>
             </visual>
             <collision>
@@ -71,5 +71,5 @@
                     <mesh filename="file://$(arg models_dir)/cyton/meshes/visual/link2.dae" />
                 </geometry>
-                <material name="blue"/>
+                <material name="TopBlack"/>
             </visual>
             <collision>
@@ -102,5 +102,5 @@
                     <mesh filename="file://$(arg models_dir)/cyton/meshes/visual/link3.dae" />
                 </geometry>
-                <material name="blue"/>
+                <material name="TopBlack"/>
             </visual>
             <collision>
@@ -134,5 +134,5 @@
                     <mesh filename="file://$(arg models_dir)/cyton/meshes/visual/link4.dae" />
                 </geometry>
-                <material name="blue"/>
+                <material name="TopBlack"/>
             </visual>
             <collision>
@@ -165,5 +165,5 @@
                     <mesh filename="file://$(arg models_dir)/cyton/meshes/visual/link5.dae" />
                 </geometry>
-                <material name="blue"/>
+                <material name="TopBlack"/>
             </visual>
             <collision>
@@ -196,5 +196,5 @@
                     <mesh filename="file://$(arg models_dir)/cyton/meshes/visual/link6.dae" />
                 </geometry>
-                <material name="blue"/>
+                <material name="TopBlack"/>
             </visual>
             <collision>
@@ -227,5 +227,5 @@
                     <mesh filename="file://$(arg models_dir)/cyton/meshes/visual/link7.dae" />
                 </geometry>
-                <material name="blue"/>
+                <material name="TopBlack"/>
             </visual>
             <collision>
@@ -266,5 +266,5 @@
                     <mesh filename="file://$(arg models_dir)/cyton/meshes/visual/link8.dae" scale="1.0 1.0 2.0"/>
                 </geometry>
-                <material name="blue"/>
+                <material name="TopBlack"/>
             </visual>
             <collision>
@@ -297,5 +297,5 @@
                     <mesh filename="file://$(arg models_dir)/cyton/meshes/visual/link9.dae" scale="1.0 1.0 2.0"/>
                 </geometry>
-                <material name="blue"/>
+                <material name="TopBlack"/>
             </visual>
             <collision>

File: src/mobile_arm_description/description/materials.xacro (robot description, xacro)
@@ -31,3 +31,6 @@
     <color rgba="1.0 1.0 1.0 1.0"/>
   </material>
+  <material name="TopBlack">
+    <color rgba="0.038 0.038 0.038 1.0"/>
+  </material>
 </robot>
