Commit message: hardware plugins added

File: src/mobile_arm_description/description/pioneer3dx/main.xacro (robot description, xacro)
@@ -11,4 +11,6 @@
   <xacro:arg name="laser0_driver"    default="gpu"/>
   <xacro:arg name="use_sim"          default="False"/>
+  <xacro:arg name="usb_port"         default="/dev/ttyUSB0"/>
+  <xacro:arg name="baud_rate"        default="115200"/>
   <xacro:arg name="initial_positions_file"      default="$(find mobile_arm_moveit)/config/initial_positions.yaml"/>
   <xacro:property name="models_dir"    value="$(arg models_dir)"/>
@@ -26,8 +28,8 @@
   <xacro:include filename="${models_dir}/${robot_model}/plugins_hardware.xacro"/>
   <xacro:if value="$(arg use_sim)">
-    <xacro:plugins_ignition />
+    <xacro:plugins_ignition/>
   </xacro:if>
   <xacro:unless value="$(arg use_sim)">
-    <xacro:plugins_hardware initial_positions_file="$(arg initial_positions_file)"/>
+    <xacro:plugins_hardware usb_port="${usb_port}" baud_rate="${baud_rate}" initial_positions_file="$(arg initial_positions_file)"/>
   </xacro:unless>
   <!-- Laser -->

File: src/mobile_arm_description/description/pioneer3dx/plugins_hardware.xacro (robot description, xacro)
@@ -1,11 +1,12 @@
 <?xml version="1.0"?>
 <robot xmlns:xacro="http://ros.org/wiki/xacro">
-    <xacro:macro name="plugins_hardware" params="initial_positions_file">
-      <xacro:property name="initial_positions" value="${xacro.load_yaml(initial_positions_file)['initial_positions']}"/>
+    <xacro:macro name="plugins_hardware" params="usb_port baud_rate initial_positions_file">
+        <xacro:macro name="ros_control_dynamixel" params="usb_port baud_rate">
+        <xacro:property name="initial_positions" value="${xacro.load_yaml(initial_positions_file)['initial_positions']}"/>
         <ros2_control name="DynamixelHardware" type="system">
             <hardware>
               <plugin>dynamixel_hardware/DynamixelHardware</plugin>
-              <param name="usb_port">/dev/ttyUSB0</param>
-              <param name="baud_rate">115200</param>
+              <param name="usb_port">${usb_port}</param>
+              <param name="baud_rate">${baud_rate}</param>
               <param name="joint_ids">1,2,3,4,5,6,7,8</param>
             </hardware>
@@ -76,4 +77,40 @@
             </joint>
         </ros2_control>
+      </xacro:macro>
+      <xacro:macro name="ros_control_odrive" params="name">
+        <ros2_control name="${name}_motors" type="system">
+            <hardware>
+              <plugin>???PioneerDriver???</plugin>
+              <param name="velocity_limit">30</param>
+              <param name="current_limit">60</param>
+            </hardware>
+          <joint name="left_wheel_joint">
+              <command_interface name="velocity">
+                  <param name="min">-10</param>
+                  <param name="max">10</param>
+              </command_interface>
+              <state_interface name="velocity"/>
+              <state_interface name="position"/>
+          </joint>
+          <joint name="right_wheel_joint">
+              <command_interface name="velocity">
+                  <param name="min">-10</param>
+                  <param name="max">10</param>
+              </command_interface>
+              <state_interface name="velocity"/>
+              <state_interface name="position"/>
+          </joint>
+          <joint name="swivel_joint">
+              <state_interface name="velocity"/>
+              <state_interface name="position"/>
+          </joint>
+          <joint name="swivel_wheel_joint">
+              <state_interface name="velocity"/>
+              <state_interface name="position"/>
+          </joint>
+        </ros2_control>
+      </xacro:macro>
+      <xacro:ros_control_dynamixel usb_port="${usb_port}" baud_rate="${baud_rate}" />
+      <xacro:ros_control_odrive name="pioneer"/>
     </xacro:macro>
 <!-- insert ros2 hardware controllers here -->

File: src/mobile_arm_description/description/pioneer3dx/plugins_ignition.xacro (robot description, xacro)
@@ -130,17 +130,4 @@
           </plugin>
       </gazebo>
-      <!-- <gazebo>
-      <plugin name="gazebo_ros_joint_state_publisher"
-          filename="libgazebo_ros_joint_state_publisher.so">
-        <ros>
-          <remapping>joint_states:=joint_states</remapping>
-        </ros>
-        <update_rate>10</update_rate>
-        <joint_name>left_wheel_joint</joint_name>
-        <joint_name>right_wheel_joint</joint_name>
-        <joint_name>swivel_joint</joint_name>
-        <joint_name>swivel_wheel_joint</joint_name>
-      </plugin>
-      </gazebo>     -->
   </xacro:macro>
 </robot>

Commit message: lab1.5

File: src/mobile_arm_description/description/pioneer3dx/main.xacro (robot description, xacro)
@@ -39,5 +39,5 @@
   <!-- Arm -->
   <xacro:include filename="${models_dir}/${arm_model}/main.xacro" />
-  <xacro:arm name="cyton" parent="top" xyz="0.088 -0.02 0.005" rpy="0 0 0" use_sim="$(arg use_sim)"/>
+  <xacro:arm name="cyton" parent="top" xyz="0.109 0.0 -0.016" rpy="0 0 1.5707" use_sim="$(arg use_sim)"/>
   <!-- <xacro:arm name="cyton" parent="top" xyz="0.0 0.0 0.0" rpy="0 0 0" use_sim="$(arg use_sim)"/> -->
 </robot>

File: src/mobile_arm_description/description/pioneer3dx/plugins_hardware.xacro (robot description, xacro)
@@ -78,39 +78,5 @@
         </ros2_control>
       </xacro:macro>
-      <xacro:macro name="ros_control_odrive" params="name">
-        <ros2_control name="${name}_motors" type="system">
-            <hardware>
-              <plugin>???PioneerDriver???</plugin>
-              <param name="velocity_limit">30</param>
-              <param name="current_limit">60</param>
-            </hardware>
-          <joint name="left_wheel_joint">
-              <command_interface name="velocity">
-                  <param name="min">-10</param>
-                  <param name="max">10</param>
-              </command_interface>
-              <state_interface name="velocity"/>
-              <state_interface name="position"/>
-          </joint>
-          <joint name="right_wheel_joint">
-              <command_interface name="velocity">
-                  <param name="min">-10</param>
-                  <param name="max">10</param>
-              </command_interface>
-              <state_interface name="velocity"/>
-              <state_interface name="position"/>
-          </joint>
-          <joint name="swivel_joint">
-              <state_interface name="velocity"/>
-              <state_interface name="position"/>
-          </joint>
-          <joint name="swivel_wheel_joint">
-              <state_interface name="velocity"/>
-              <state_interface name="position"/>
-          </joint>
-        </ros2_control>
-      </xacro:macro>
       <xacro:ros_control_dynamixel usb_port="${usb_port}" baud_rate="${baud_rate}" />
-      <xacro:ros_control_odrive name="pioneer"/>
     </xacro:macro>
 <!-- insert ros2 hardware controllers here -->
