Commit message: testing

File: src/mobile_arm_description/description/pioneer3dx/body copy/swivel.xacro (robot description, xacro)
@@ -4,5 +4,5 @@
   <xacro:macro name="pioneer_swivel" params="name parent xyz rpy models_dir:=^ ">
   <!-- Swivel -->
-  <joint name="${name}_joint" type="fixed">
+  <joint name="${name}_joint" type="continuous">
     <origin xyz="${xyz}" rpy="${rpy}"/>
     <axis xyz="0 0 1"/>
@@ -43,5 +43,5 @@
   </gazebo>
   <!-- Center Wheel -->
-  <joint name="${name}_wheel_joint" type="fixed">
+  <joint name="${name}_wheel_joint" type="continuous">
     <origin xyz="-0.026 0 -0.016" rpy="0 0 0"/>
     <axis xyz="0 1 0" />

File: src/mobile_arm_description/description/pioneer3dx/body copy/wheel.xacro (robot description, xacro)
@@ -4,8 +4,10 @@
   <xacro:macro name="pioneer_wheel" params="name parent xyz rpy radius models_dir:=^">
     <!-- Wheel -->
-    <joint name="${name}_wheel_joint" type="fixed">
+    <joint name="${name}_wheel_joint" type="continuous">
 		<origin xyz="${xyz}" rpy="${rpy}"/>
 		<parent link="${parent}"/>
 		<child link="${name}_wheel"/>
+		<axis xyz="0 1 0"/>
+		<dynamics damping="0.2" friction="0.7"/>
     </joint>
     <link name="${name}_wheel">
