Commit message: simulation problem

File: src/mobile_arm_description/description/pioneer3dx/body copy/body.xacro (robot description, xacro)
@@ -19,5 +19,5 @@
     <xacro:pioneer_battery_block name="battery0" parent="${name}" x="-0.14" y="0.00"  z="${0.13-0.068}" mass="5.5" />
     <!-- Wheels -->
-    <xacro:property name="contact_data">
+    <!-- <xacro:property name="contact_data">
         <mu1 value="0.7"/>
         <mu2 value="0.7"/>
@@ -25,5 +25,5 @@
         <kp value="1000000.0"/>
         <kd value="10.0"/>
-    </xacro:property>
+    </xacro:property>  -->
     <!-- Swivels -->
     <xacro:pioneer_swivel  name="swivel"    parent="${parent}"  xyz="-0.185 0    0.0555" rpy="0 0 0"/>

File: src/mobile_arm_description/description/pioneer3dx/body copy/swivel.xacro (robot description, xacro)
@@ -4,7 +4,10 @@
   <xacro:macro name="pioneer_swivel" params="name parent xyz rpy models_dir:=^ ">
   <!-- Swivel -->
-  <joint name="${name}_joint" type="fixed">
+  <joint name="${name}_joint" type="continuous">
     <origin xyz="${xyz}" rpy="${rpy}"/>
+    <axis xyz="0 0 1"/>
     <anchor xyz="0 0 0"/>
+    <limit effort="100" velocity="100" k_velocity="0"/>
+    <joint_properties damping="0.1" friction="0.0"/>
     <parent link="${parent}"/>
     <child link="${name}"/>
@@ -40,6 +43,7 @@
   </gazebo>
   <!-- Center Wheel -->
-  <joint name="${name}_wheel_joint" type="fixed">
+  <joint name="${name}_wheel_joint" type="continuous">
     <origin xyz="-0.026 0 -0.016" rpy="0 0 0"/>
+    <axis xyz="0 1 0" />
     <anchor xyz="0 0 0"/>
     <parent link="${name}"/>
