Commit message: działa czasami

File: src/mobile_arm_description/description/pioneer3dx/body_nodiff/swivel.xacro (robot description, xacro)
@@ -4,5 +4,5 @@
   <xacro:macro name="pioneer_swivel" params="name parent xyz rpy models_dir:=^ ">
   <!-- Swivel -->
-  <joint name="${name}_joint" type="continuous">
+  <joint name="${name}_joint" type="fixed">
     <origin xyz="${xyz}" rpy="${rpy}"/>
     <axis xyz="0 0 1"/>
@@ -43,5 +43,5 @@
   </gazebo>
   <!-- Center Wheel -->
-  <joint name="${name}_wheel_joint" type="continuous">
+  <joint name="${name}_wheel_joint" type="fixed">
     <origin xyz="-0.026 0 -0.016" rpy="0 0 0"/>
     <axis xyz="0 1 0" />

File: src/mobile_arm_description/description/pioneer3dx/body_nodiff/wheel.xacro (robot description, xacro)
@@ -4,10 +4,8 @@
   <xacro:macro name="pioneer_wheel" params="name parent xyz rpy radius models_dir:=^">
     <!-- Wheel -->
-    <joint name="${name}_wheel_joint" type="continuous">
+    <joint name="${name}_wheel_joint" type="fixed">
 		<origin xyz="${xyz}" rpy="${rpy}"/>
 		<parent link="${parent}"/>
 		<child link="${name}_wheel"/>
-		<axis xyz="0 1 0"/>
-		<dynamics damping="0.2" friction="0.7"/>
     </joint>
     <link name="${name}_wheel">

File: src/mobile_arm_description/description/pioneer3dx/main.xacro (robot description, xacro)
@@ -39,5 +39,5 @@
   <!-- Arm -->
   <xacro:include filename="${models_dir}/${arm_model}/main.xacro" />
-  <xacro:arm name="cyton" parent="top" xyz="0.26 0.0 -0.16" rpy="0 0 1.5707" use_sim="$(arg use_sim)"/>
+  <xacro:arm name="cyton" parent="top" xyz="0.26 0.0 -0.16" rpy="0 0 3.1415" use_sim="$(arg use_sim)"/>
   <!-- <xacro:arm name="cyton" parent="top" xyz="0.0 0.0 0.0" rpy="0 0 0" use_sim="$(arg use_sim)"/> -->
 </robot>
